File: kicad/matter-plant-sensor/_autosave-matter-plant-sensor.kicad_sch (KiCad schematic)
At the start: 6 parts, among them SW1 SW_Push, U1 ESP32-H2-SUPERMINI, U2 BH1750_Module, U3 SHT41_Module

Commit message: Setup kicad schematics
Parts:
- added U4: TP4056_Module, symbol Sensor_Custom:TP4056_Module
Changed lines of the file:
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@@
+	)
+	(symbol
+		(lib_id "Sensor_Custom:TP4056_Module")
+		(at 193.04 134.62 0)
+		(unit 1)
+		(exclude_from_sim no)
+		(in_bom yes)
+		(on_board yes)
+		(dnp no)
+		(fields_autoplaced yes)
+		(property "Reference" "U4"
+			(at 195.1833 121.92 0)
+			(effects
+				(font
+					(size 1.27 1.27)
+				)
+				(justify left)
+			)
+		)
+		(property "Value" "TP4056_Module"
+			(at 195.1833 124.46 0)
+			(effects
+				(font
+					(size 1.27 1.27)
+				)
+				(justify left)
+			)
+		)
+		(property "Footprint" ""
+			(at 193.04 134.62 0)
+			(effects
+				(font
+					(size 1.27 1.27)
+				)
+				(hide yes)
+			)
+		)
+		(property "Datasheet" ""
+			(at 193.04 134.62 0)
+			(effects
+				(font
+					(size 1.27 1.27)
+				)
+				(hide yes)
+			)
+		)
+		(property "Description" ""
+			(at 193.04 134.62 0)
+			(effects
+				(font
+					(size 1.27 1.27)
+				)
+				(hide yes)
+			)
+		)
+		(pin "3"
+		)
+		(pin "1"
+		)
+		(pin "4"
+		)
+		(pin "2"
+		)
+		(pin "5"
+		)
+		(pin "6"
+		)
+		(instances
+			(project ""
+				(path "/19d6e18f-c506-4214-a7b7-d6af9c07898d"
+					(reference "U4")
+					(unit 1)
+				)
+			)
+		)
 	)
 	(symbol
